File: optical-keyboard.kicad_pcb (KiCad board)
At the start: 2 copper layers, 11 x 32.5 mm, 472 parts, among them Q1 Q_Photo_NPN, Q10 Q_Photo_NPN, Q11 Q_Photo_NPN, Q12 Q_Photo_NPN, Q13 Q_Photo_NPN, Q14 Q_Photo_NPN, Q15 Q_Photo_NPN, Q16 Q_Photo_NPN, Q17 Q_Photo_NPN, Q18 Q_Photo_NPN, Q19 Q_Photo_NPN, Q2 Q_Photo_NPN, Q20 Q_Photo_NPN, Q21 Q_Photo_NPN, Q22 Q_Photo_NPN, Q23 Q_Photo_NPN, Q24 Q_Photo_NPN, Q25 Q_Photo_NPN, Q26 Q_Photo_NPN, Q27 Q_Photo_NPN, Q28 Q_Photo_NPN, Q29 Q_Photo_NPN, Q3 Q_Photo_NPN, Q30 Q_Photo_NPN, Q31 Q_Photo_NPN, Q32 Q_Photo_NPN, Q33 Q_Photo_NPN, Q34 Q_Photo_NPN, Q35 Q_Photo_NPN, Q36 Q_Photo_NPN, Q37 Q_Photo_NPN, Q38 Q_Photo_NPN, Q39 Q_Photo_NPN, Q4 Q_Photo_NPN, Q40 Q_Photo_NPN, Q41 Q_Photo_NPN, Q42 Q_Photo_NPN, Q43 Q_Photo_NPN, Q44 Q_Photo_NPN, Q45 Q_Photo_NPN, Q46 Q_Photo_NPN, Q47 Q_Photo_NPN, Q48 Q_Photo_NPN, Q49 Q_Photo_NPN, Q5 Q_Photo_NPN, Q50 Q_Photo_NPN, Q51 Q_Photo_NPN, Q52 Q_Photo_NPN, Q53 Q_Photo_NPN, Q54 Q_Photo_NPN, Q55 Q_Photo_NPN, Q56 Q_Photo_NPN, Q57 Q_Photo_NPN, Q58 Q_Photo_NPN, Q59 Q_Photo_NPN, Q6 Q_Photo_NPN, Q60 Q_Photo_NPN, Q61 Q_Photo_NPN, Q62 Q_Photo_NPN, Q63 Q_Photo_NPN, Q64 Q_Photo_NPN, Q65 Q_Photo_NPN, Q66 Q_Photo_NPN, Q67 Q_Photo_NPN, Q68 Q_Photo_NPN, Q69 Q_Photo_NPN, Q7 Q_Photo_NPN, Q70 Q_Photo_NPN, Q71 Q_Photo_NPN, Q72 Q_Photo_NPN, Q73 Q_Photo_NPN, Q74 Q_Photo_NPN, Q75 Q_Photo_NPN, Q8 Q_Photo_NPN, Q9 Q_Photo_NPN, U1 BlackPill_STLINK

Commit message: updated pcb
M  optical-keyboard.kicad_pcb
M  optical-keyboard.kicad_pro
M  optical-keyboard.kicad_sch
M  placefp.py
M  switch.kicad_sch
Parts:
- added H20: MountingHole, OpticalParts:TestPoint_Plated_Hole_D1.2mm, F.Cu at (7.14, 47.6)
- H16: footprint OpticalParts:TestPoint_Plated_Hole_D1.2mm -> OpticalParts:MountingHole_2.2mm_M2_jlcpcb
- N1, N10, N11, N12, N13, N14, N15, N16, N17, N18, N19, N2, N20, N21, N22, N23, N24, N25, N26, N27, N28, N29, N3, N30, N31, N32, N33, N34, N35, N36, N37, N38, N39, N4, N40, N41, N42, N43, N44, N45, N46, N47, N48, N49, N5, N50, N51, N52, N53, N54, N55, N56, N57, N58, N59, N6, N60, N61, N62, N63, N64, N65, N66, N67, N68, N69, N7, N70, N71, N72, N73, N74, N75, N8, N9: footprint Diode_SMD:D_SOD-323 -> Diode_SMD:D_SOD-323_HandSoldering
- moved Q31 531.0 mm to (12.9, 38.1)
- moved RL31 525.8 mm to (17.8, 42.1)
- moved S31 520.4 mm to (9.53, 38.1)
- moved D31 514.2 mm to (6.12, 38.1)
- moved N31 506.9 mm to (17.8, 34.1), turned to -90 degrees
- moved RP31 501.7 mm to (17.8, 38.1)
- moved Q47 378.8 mm to (46.3, 57.1)
- moved Q19 377.1 mm to (89.1, 19.1)
- moved RL47 374.0 mm to (51.2, 61.1)
- moved RL19 371.5 mm to (94.0, 23.1)
- moved S19 368.4 mm to (85.7, 19.1)
- moved S47 367.5 mm to (42.9, 57.1)
- moved Q39 366.6 mm to (170.1, 38.1)
- moved D19 365.8 mm to (82.3, 19.1)
- moved RL39 361.3 mm to (175.0, 42.1)
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Connections:
- U1 pad 44: GND -> unconnected-(U1-Pad44)
Routing:
- net /col15: track 0.00 -> 442.3 mm, vias 0 -> 10
- net /row2: track 0.00 -> 356.8 mm, vias 0 -> 3
- net /row1: track 0.00 -> 353.6 mm, vias 0 -> 2
- net /col14: track 0.00 -> 351.7 mm, vias 0 -> 9
- net /row5: track 0.00 -> 345.6 mm, vias 0 -> 1
- net /col13: track 0.00 -> 328.5 mm, vias 0 -> 9
- net GND: track 0.00 -> 317.2 mm, vias 0 -> 153
- net /col12: track 0.00 -> 312.7 mm, vias 0 -> 9
- net /row4: track 0.00 -> 304.8 mm, vias 0 -> 1
- net /row3: track 0.00 -> 298.7 mm, vias 0 -> 1
- net /col11: track 0.00 -> 296.8 mm, vias 0 -> 9
- net /col10: track 0.00 -> 281.5 mm, vias 0 -> 9
- net /col9: track 0.00 -> 262.2 mm, vias 0 -> 9
- net /col8: track 0.00 -> 242.5 mm, vias 0 -> 9
- net /col7: track 0.00 -> 232.5 mm, vias 0 -> 9
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- added copper zone on B.Cu, net GND
Other:
- board size 11 x 32.5 mm -> 304.8 x 114.3 mm
