File: optical-keyboard.kicad_pcb (KiCad board)
At the start: 2 copper layers, 304.8 x 114.3 mm, 473 parts, among them Q1 Q_Photo_NPN, Q10 Q_Photo_NPN, Q11 Q_Photo_NPN, Q12 Q_Photo_NPN, Q13 Q_Photo_NPN, Q14 Q_Photo_NPN, Q15 Q_Photo_NPN, Q16 Q_Photo_NPN, Q17 Q_Photo_NPN, Q18 Q_Photo_NPN, Q19 Q_Photo_NPN, Q2 Q_Photo_NPN, Q20 Q_Photo_NPN, Q21 Q_Photo_NPN, Q22 Q_Photo_NPN, Q23 Q_Photo_NPN, Q24 Q_Photo_NPN, Q25 Q_Photo_NPN, Q26 Q_Photo_NPN, Q27 Q_Photo_NPN, Q28 Q_Photo_NPN, Q29 Q_Photo_NPN, Q3 Q_Photo_NPN, Q30 Q_Photo_NPN, Q31 Q_Photo_NPN, Q32 Q_Photo_NPN, Q33 Q_Photo_NPN, Q34 Q_Photo_NPN, Q35 Q_Photo_NPN, Q36 Q_Photo_NPN, Q37 Q_Photo_NPN, Q38 Q_Photo_NPN, Q39 Q_Photo_NPN, Q4 Q_Photo_NPN, Q40 Q_Photo_NPN, Q41 Q_Photo_NPN, Q42 Q_Photo_NPN, Q43 Q_Photo_NPN, Q44 Q_Photo_NPN, Q45 Q_Photo_NPN, Q46 Q_Photo_NPN, Q47 Q_Photo_NPN, Q48 Q_Photo_NPN, Q49 Q_Photo_NPN, Q5 Q_Photo_NPN, Q50 Q_Photo_NPN, Q51 Q_Photo_NPN, Q52 Q_Photo_NPN, Q53 Q_Photo_NPN, Q54 Q_Photo_NPN, Q55 Q_Photo_NPN, Q56 Q_Photo_NPN, Q57 Q_Photo_NPN, Q58 Q_Photo_NPN, Q59 Q_Photo_NPN, Q6 Q_Photo_NPN, Q60 Q_Photo_NPN, Q61 Q_Photo_NPN, Q62 Q_Photo_NPN, Q63 Q_Photo_NPN, Q64 Q_Photo_NPN, Q65 Q_Photo_NPN, Q66 Q_Photo_NPN, Q67 Q_Photo_NPN, Q68 Q_Photo_NPN, Q69 Q_Photo_NPN, Q7 Q_Photo_NPN, Q70 Q_Photo_NPN, Q71 Q_Photo_NPN, Q72 Q_Photo_NPN, Q73 Q_Photo_NPN, Q74 Q_Photo_NPN, Q75 Q_Photo_NPN, Q8 Q_Photo_NPN, Q9 Q_Photo_NPN, U1 BlackPill_STLINK

Commit message: Add separate power source for PTs
Sharing input pin b/w pt and led requires a diode, and diode
slows down the response time of pt considerably

M  optical-keyboard.kicad_pcb
M  optical-keyboard.kicad_prl
M  optical-keyboard.kicad_sch
M  placefp.py
M  switch.kicad_sch
Parts:
- removed N1, N10, N11, N12, N13, N14, N15, N16, N17, N18, N19, N2, N20, N21, N22, N23, N24, N25, N26, N27, N28, N29, N3, N30, N31, N32, N33, N34, N35, N36, N37, N38, N39, N4, N40, N41, N42, N43, N44, N45, N46, N47, N48, N49, N5, N50, N51, N52, N53, N54, N55, N56, N57, N58, N59, N6, N60, N61, N62, N63, N64, N65, N66, N67, N68, N69, N7, N70, N71, N72, N73, N74, N75, N8, N9: Diode1N4148WSSod323, Diode_SMD:D_SOD-323_HandSoldering
- removed RP10, RP11, RP12, RP13, RP14, RP15, RP16, RP17, RP18, RP19, RP20, RP21, RP22, RP23, RP24, RP25, RP26, RP27, RP28, RP29, RP30, RP31, RP32, RP33, RP34, RP35, RP36, RP37, RP38, RP39, RP40, RP41, RP42, RP43, RP44, RP45, RP46, RP47, RP48, RP49, RP50, RP51, RP52, RP53, RP54, RP55, RP56, RP57, RP58, RP59, RP6, RP60, RP61, RP62, RP63, RP64, RP65, RP66, RP67, RP68, RP69, RP7, RP70, RP71, RP72, RP73, RP74, RP75, RP8, RP9: R_PT, Resistor_SMD:R_0805_2012Metric
- moved RP5 80.1 mm to (77.4, 75.7)
- moved RP1 57.2 mm to (84.5, -0.50)
- moved RP4 56.8 mm to (89.3, 56.6)
- moved RP2 51.1 mm to (94.0, 18.6)
- moved RP3 40.2 mm to (79.7, 37.6)
Connections:
- Q1 pad 1: Net-(N1-Pad2) -> /row1
- Q10 pad 1: Net-(N10-Pad2) -> /row1
- Q11 pad 1: Net-(N11-Pad2) -> /row1
- Q12 pad 1: Net-(N12-Pad2) -> /row1
- Q13 pad 1: Net-(N13-Pad2) -> /row1
- Q14 pad 1: Net-(N14-Pad2) -> /row1
- Q15 pad 1: Net-(N15-Pad2) -> /row1
- Q16 pad 1: Net-(N16-Pad2) -> /row2
- Q17 pad 1: Net-(N17-Pad2) -> /row2
- Q18 pad 1: Net-(N18-Pad2) -> /row2
- Q19 pad 1: Net-(N19-Pad2) -> /row2
- Q2 pad 1: Net-(N2-Pad2) -> /row1
- Q20 pad 1: Net-(N20-Pad2) -> /row2
- Q21 pad 1: Net-(N21-Pad2) -> /row2
- Q22 pad 1: Net-(N22-Pad2) -> /row2
- Q23 pad 1: Net-(N23-Pad2) -> /row2
- Q24 pad 1: Net-(N24-Pad2) -> /row2
- Q25 pad 1: Net-(N25-Pad2) -> /row2
- Q26 pad 1: Net-(N26-Pad2) -> /row2
- Q27 pad 1: Net-(N27-Pad2) -> /row2
- Q28 pad 1: Net-(N28-Pad2) -> /row2
- Q29 pad 1: Net-(N29-Pad2) -> /row2
- Q3 pad 1: Net-(N3-Pad2) -> /row1
- Q30 pad 1: Net-(N30-Pad2) -> /row2
- Q31 pad 1: Net-(N31-Pad2) -> /row3
- Q32 pad 1: Net-(N32-Pad2) -> /row3
- Q33 pad 1: Net-(N33-Pad2) -> /row3
- Q34 pad 1: Net-(N34-Pad2) -> /row3
- Q35 pad 1: Net-(N35-Pad2) -> /row3
- Q36 pad 1: Net-(N36-Pad2) -> /row3
- Q37 pad 1: Net-(N37-Pad2) -> /row3
- Q38 pad 1: Net-(N38-Pad2) -> /row3
- Q39 pad 1: Net-(N39-Pad2) -> /row3
- Q4 pad 1: Net-(N4-Pad2) -> /row1
- Q40 pad 1: Net-(N40-Pad2) -> /row3
- Q41 pad 1: Net-(N41-Pad2) -> /row3
- Q42 pad 1: Net-(N42-Pad2) -> /row3
- Q43 pad 1: Net-(N43-Pad2) -> /row3
- Q44 pad 1: Net-(N44-Pad2) -> /row3
- Q45 pad 1: Net-(N45-Pad2) -> /row3
- Q46 pad 1: Net-(N46-Pad2) -> /row4
- Q47 pad 1: Net-(N47-Pad2) -> /row4
- Q48 pad 1: Net-(N48-Pad2) -> /row4
- Q49 pad 1: Net-(N49-Pad2) -> /row4
- Q5 pad 1: Net-(N5-Pad2) -> /row1
- Q50 pad 1: Net-(N50-Pad2) -> /row4
- Q51 pad 1: Net-(N51-Pad2) -> /row4
- Q52 pad 1: Net-(N52-Pad2) -> /row4
- Q53 pad 1: Net-(N53-Pad2) -> /row4
- Q54 pad 1: Net-(N54-Pad2) -> /row4
- Q55 pad 1: Net-(N55-Pad2) -> /row4
- Q56 pad 1: Net-(N56-Pad2) -> /row4
- Q57 pad 1: Net-(N57-Pad2) -> /row4
- Q58 pad 1: Net-(N58-Pad2) -> /row4
- Q59 pad 1: Net-(N59-Pad2) -> /row4
- Q6 pad 1: Net-(N6-Pad2) -> /row1
- Q60 pad 1: Net-(N60-Pad2) -> /row4
- Q61 pad 1: Net-(N61-Pad2) -> /row5
- Q62 pad 1: Net-(N62-Pad2) -> /row5
- Q63 pad 1: Net-(N63-Pad2) -> /row5
- Q64 pad 1: Net-(N64-Pad2) -> /row5
- Q65 pad 1: Net-(N65-Pad2) -> /row5
- Q66 pad 1: Net-(N66-Pad2) -> /row5
- Q67 pad 1: Net-(N67-Pad2) -> /row5
- Q68 pad 1: Net-(N68-Pad2) -> /row5
- Q69 pad 1: Net-(N69-Pad2) -> /row5
- Q7 pad 1: Net-(N7-Pad2) -> /row1
- Q70 pad 1: Net-(N70-Pad2) -> /row5
- Q71 pad 1: Net-(N71-Pad2) -> /row5
- Q72 pad 1: Net-(N72-Pad2) -> /row5
- Q73 pad 1: Net-(N73-Pad2) -> /row5
- Q74 pad 1: Net-(N74-Pad2) -> /row5
- Q75 pad 1: Net-(N75-Pad2) -> /row5
- Q8 pad 1: Net-(N8-Pad2) -> /row1
- Q9 pad 1: Net-(N9-Pad2) -> /row1
- RP1 pad 1: /col1 -> /row1
- RP1 pad 2: Net-(N1-Pad2) -> 3v3
- RP2 pad 1: /col2 -> /row2
- RP2 pad 2: Net-(N2-Pad2) -> 3v3
- RP3 pad 1: /col3 -> /row3
- RP3 pad 2: Net-(N3-Pad2) -> 3v3
- RP4 pad 1: /col4 -> /row4
- RP4 pad 2: Net-(N4-Pad2) -> 3v3
- RP5 pad 1: /col5 -> /row5
- RP5 pad 2: Net-(N5-Pad2) -> 3v3
- U1 pad 20: unconnected-(U1-Pad20) -> 3v3
- U1 pad 3: /row1 -> /row3
- U1 pad 35: /col4 -> /col1
- U1 pad 37: /col1 -> /row1
- U1 pad 4: /row3 -> /col4
Routing:
- net 3v3: track 0.00 -> 146.4 mm, vias 0 -> 7
- net /col1: track 186.1 -> 115.9 mm, vias 9 -> 7
- net /row1: track 353.6 -> 311.7 mm, vias 2 -> 1
- net /row5: track 345.6 -> 379.6 mm
- net /row4: track 304.8 -> 337.9 mm
- net /row2: track 356.8 -> 380.7 mm
- net /row3: track 298.7 -> 320.2 mm, vias 1 -> 0
- net /col15: track 442.3 -> 461.7 mm, vias 10 -> 7
- net /col2: track 137.0 -> 127.1 mm, vias 9 -> 6
- net GND: track 317.2 -> 307.3 mm, vias 153 -> 151
- net /col6: track 216.1 -> 207.7 mm, vias 8 -> 6
- net Net-(N45-Pad2): track 6.98 -> 0.00 mm
- net Net-(N67-Pad2): track 6.98 -> 0.00 mm
- net Net-(N46-Pad2): track 6.80 -> 0.00 mm
- net Net-(N54-Pad2): track 6.80 -> 0.00 mm
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Other:
- outline, holes or cut-outs redrawn
